Commit message: updated urdf

File: test/urdf/macro_old.xacro (robot description, xacro)
@@ -30,4 +30,5 @@
         <origin xyz="0 0 0" rpy="0 0 0"/>
       </joint>
+    </xacro:macro>
   <!-- Prismatic joint 1 -->
   <xacro:macro name="link2" params="l1">

File: test_1/urdf/scara_urdf.xacro (robot description, xacro)
@@ -1,12 +1,11 @@
 <?xml version="1.0"?>
 <robot name="scara" xmlns:xacro="http://www.ros.org/wiki/xacro">
-  <!-- === Parameters === -->
-  <xacro:property name="link_2_length" value="0.45"/>
-  <xacro:property name="link_2_radius" value="0.05"/>
-  <xacro:property name="link_3_length" value="0.425"/>
-  <xacro:property name="link_4_length" value="0.2"/>
-  <xacro:property name="link_4_radius" value="0.05"/>
-  <xacro:property name="link_5_length" value="0.345"/>
-  <!-- === Materials === -->
+  <xacro:property name="l2" value="0.45"/>
+  <xacro:property name="l2_r" value="0.05"/>
+  <xacro:property name="l3" value="0.425"/>
+  <xacro:property name="l4" value="0.2"/>
+  <xacro:property name="l4_r" value="0.05"/>
+  <xacro:property name="l5" value="0.345"/>
+  <xacro:property name="gripper_length" value="0.1"/>
   <material name="blue">
     <color rgba="0 0 1 1"/>
@@ -18,5 +17,5 @@
     <color rgba="0 1 0 1"/>
   </material>
-  <!-- === Links === -->
+<!--links-->
   <link name="base_link"/>
   <link name="link_1">
@@ -37,12 +36,12 @@
     <visual>
       <geometry>
-        <cylinder length="${link_2_length}" radius="${link_2_radius}"/>
+        <cylinder length="${l2}" radius="${l2_r}"/>
       </geometry>
       <material name="blue"/>
-      <origin xyz="0 0 ${link_2_length/2}"/>
+      <origin xyz="0 0 ${l2/2}"/>
     </visual>
     <inertial>
       <mass value="0.5"/>
-      <origin xyz="0 0 ${link_2_length/2}"/>
+      <origin xyz="0 0 ${l2/2}"/>
       <inertia ixx="0.5" ixy="0" ixz="0" iyy="0.5" iyz="0" izz="0.5"/>
     </inertial>
@@ -51,12 +50,12 @@
     <visual>
       <geometry>
-        <box size="0.1 0.1 ${link_3_length}"/>
+        <box size="0.1 0.1 ${l3}"/>
       </geometry>
       <material name="red"/>
-      <origin rpy="0 1.571 0" xyz="${link_3_length/2} 0 0"/>
+      <origin rpy="0 1.571 0" xyz="${l3/2} 0 0"/>
     </visual>
     <inertial>
       <mass value="0.5"/>
-      <origin xyz="${link_3_length/2} 0 0"/>
+      <origin xyz="${l3/2} 0 0"/>
       <inertia ixx="0.5" ixy="0" ixz="0" iyy="0.5" iyz="0" izz="0.5"/>
     </inertial>
@@ -65,5 +64,5 @@
     <visual>
       <geometry>
-        <cylinder length="${link_4_length}" radius="${link_4_radius}"/>
+        <cylinder length="${l4}" radius="${l4_r}"/>
       </geometry>
       <material name="blue"/>
@@ -79,16 +78,44 @@
     <visual>
       <geometry>
-        <box size="0.1 0.1 ${link_5_length}"/>
+        <box size="0.1 0.1 ${l5}"/>
       </geometry>
       <material name="red"/>
-      <origin rpy="0 1.571 0" xyz="${link_5_length/2} 0 0"/>
+      <origin rpy="0 1.571 0" xyz="${l5/2} 0 0"/>
     </visual>
     <inertial>
       <mass value="0.5"/>
-      <origin xyz="${link_5_length/2} 0 0"/>
+      <origin xyz="${l5/2} 0 0"/>
       <inertia ixx="0.5" ixy="0" ixz="0" iyy="0.5" iyz="0" izz="0.5"/>
     </inertial>
   </link>
-  <!-- === Fixed Joints === -->
+  <link name="link_6">
+    <inertial>
+        <origin xyz="0 0 ${l5/2}" />
+        <mass value="1"/>
+        <inertia ixx="0.1" ixy="0" ixz="0" iyy="0.1" iyz="0" izz="0.1"/>
+      </inertial>
+      <visual>
+        <origin xyz="0 0 ${l5/2}" />
+        <geometry>
+          <box size="0.1 0.1 ${l5}" />
+      </geometry>
+      <material name="green" />
+    </visual>
+  </link>
+  <link name="gripper_link">
+    <visual>
+      <origin xyz="0 0 ${-gripper_length/2}" />
+      <geometry>
+        <box size="0.08 0.08 ${gripper_length}" />
+      </geometry>
+      <material name="red"/>
+    </visual>
+    <inertial>
+      <mass value="0.2"/>
+      <origin xyz="0 0 ${-gripper_length/2}" />
+      <inertia ixx="0.1" ixy="0" ixz="0" iyy="0.1" iyz="0" izz="0.1"/>
+    </inertial>
+  </link>
+<!--Joints-->
   <joint name="fixedjoint_1" type="fixed">
     <parent link="base_link"/>
@@ -98,12 +125,17 @@
     <parent link="link_2"/>
     <child link="link_3"/>
-    <origin xyz="0 0 ${link_2_length - 0.05}"/>
+    <origin xyz="0 0 ${l2 - 0.05}"/>
   </joint>
   <joint name="fixedjoint_3" type="fixed">
     <parent link="link_4"/>
     <child link="link_5"/>
-    <origin xyz="0 0 ${link_4_length/2}"/>
+    <origin xyz="0 0 ${l4/2}"/>
   </joint>
-  <!-- === Revolute Joints === -->
+  <joint name="gripper_joint" type="fixed">
+    <parent link="link_6"/>
+    <child link="gripper_link"/>
+    <origin xyz="0 0 0" />
+  </joint>
+<!--revolut joints-->
   <joint name="revolute_1" type="revolute">
     <parent link="link_1"/>
@@ -117,8 +149,15 @@
     <parent link="link_3"/>
     <child link="link_4"/>
-    <origin xyz="${link_3_length} 0 0.05"/>
+    <origin xyz="${l3} 0 0.05"/>
     <axis xyz="0 0 1"/>
     <limit effort="1000.0" lower="-1.57" upper="1.57" velocity="0.5"/>
     <dynamics damping="0.2" friction="0.1"/>
   </joint>
+  <joint name="prismatic_joint_1" type="prismatic">
+    <parent link="link_5" />
+    <child link="link_6" />
+    <origin xyz="${l5} 0 0" rpy="0 0 0" />
+    <axis xyz="0 0 1" />
+    <limit lower="0.0" upper="${-l5}" effort="100"  velocity="1.0" />
+  </joint>
 </robot>
