Commit message: Updated scara_urdf.xacro

File: test_1/urdf/scara_urdf.xacro (robot description, xacro)
@@ -1,12 +1,10 @@
 <?xml version="1.0"?>
 <robot name="scara" xmlns:xacro="http://www.ros.org/wiki/xacro">
-  <!-- === Parameters === -->
-  <xacro:property name="link_2_length" value="0.45"/>
-  <xacro:property name="link_2_radius" value="0.05"/>
-  <xacro:property name="link_3_length" value="0.425"/>
-  <xacro:property name="link_4_length" value="0.2"/>
-  <xacro:property name="link_4_radius" value="0.05"/>
-  <xacro:property name="link_5_length" value="0.345"/>
-  <!-- === Materials === -->
+  <xacro:property name="l2" value="0.45"/>
+  <xacro:property name="l2_r" value="0.05"/>
+  <xacro:property name="l3" value="0.425"/>
+  <xacro:property name="l4" value="0.2"/>
+  <xacro:property name="l4_r" value="0.05"/>
+  <xacro:property name="l5" value="0.345"/>
   <material name="blue">
     <color rgba="0 0 1 1"/>
@@ -18,5 +16,5 @@
     <color rgba="0 1 0 1"/>
   </material>
-  <!-- === Links === -->
+<!--links-->
   <link name="base_link"/>
   <link name="link_1">
@@ -37,12 +35,12 @@
     <visual>
       <geometry>
-        <cylinder length="${link_2_length}" radius="${link_2_radius}"/>
+        <cylinder length="${l2}" radius="${l2_r}"/>
       </geometry>
       <material name="blue"/>
-      <origin xyz="0 0 ${link_2_length/2}"/>
+      <origin xyz="0 0 ${l2/2}"/>
     </visual>
     <inertial>
       <mass value="0.5"/>
-      <origin xyz="0 0 ${link_2_length/2}"/>
+      <origin xyz="0 0 ${l2/2}"/>
       <inertia ixx="0.5" ixy="0" ixz="0" iyy="0.5" iyz="0" izz="0.5"/>
     </inertial>
@@ -51,12 +49,12 @@
     <visual>
       <geometry>
-        <box size="0.1 0.1 ${link_3_length}"/>
+        <box size="0.1 0.1 ${l3}"/>
       </geometry>
       <material name="red"/>
-      <origin rpy="0 1.571 0" xyz="${link_3_length/2} 0 0"/>
+      <origin rpy="0 1.571 0" xyz="${l3/2} 0 0"/>
     </visual>
     <inertial>
       <mass value="0.5"/>
-      <origin xyz="${link_3_length/2} 0 0"/>
+      <origin xyz="${l3/2} 0 0"/>
       <inertia ixx="0.5" ixy="0" ixz="0" iyy="0.5" iyz="0" izz="0.5"/>
     </inertial>
@@ -65,5 +63,5 @@
     <visual>
       <geometry>
-        <cylinder length="${link_4_length}" radius="${link_4_radius}"/>
+        <cylinder length="${l4}" radius="${l4_r}"/>
       </geometry>
       <material name="blue"/>
@@ -79,16 +77,16 @@
     <visual>
       <geometry>
-        <box size="0.1 0.1 ${link_5_length}"/>
+        <box size="0.1 0.1 ${l5}"/>
       </geometry>
       <material name="red"/>
-      <origin rpy="0 1.571 0" xyz="${link_5_length/2} 0 0"/>
+      <origin rpy="0 1.571 0" xyz="${l5/2} 0 0"/>
     </visual>
     <inertial>
       <mass value="0.5"/>
-      <origin xyz="${link_5_length/2} 0 0"/>
+      <origin xyz="${l5/2} 0 0"/>
       <inertia ixx="0.5" ixy="0" ixz="0" iyy="0.5" iyz="0" izz="0.5"/>
     </inertial>
   </link>
-  <!-- === Fixed Joints === -->
+<!--Joints-->
   <joint name="fixedjoint_1" type="fixed">
     <parent link="base_link"/>
@@ -98,12 +96,12 @@
     <parent link="link_2"/>
     <child link="link_3"/>
-    <origin xyz="0 0 ${link_2_length - 0.05}"/>
+    <origin xyz="0 0 ${l2 - 0.05}"/>
   </joint>
   <joint name="fixedjoint_3" type="fixed">
     <parent link="link_4"/>
     <child link="link_5"/>
-    <origin xyz="0 0 ${link_4_length/2}"/>
+    <origin xyz="0 0 ${l4/2}"/>
   </joint>
-  <!-- === Revolute Joints === -->
+<!--revolut joints-->
   <joint name="revolute_1" type="revolute">
     <parent link="link_1"/>
@@ -117,5 +115,5 @@
     <parent link="link_3"/>
     <child link="link_4"/>
-    <origin xyz="${link_3_length} 0 0.05"/>
+    <origin xyz="${l3} 0 0.05"/>
     <axis xyz="0 0 1"/>
     <limit effort="1000.0" lower="-1.57" upper="1.57" velocity="0.5"/>

Commit message: Update scara_urdf.xacro

File: test_1/urdf/scara_urdf.xacro (robot description, xacro)
@@ -7,4 +7,5 @@
   <xacro:property name="l4_r" value="0.05"/>
   <xacro:property name="l5" value="0.345"/>
+  <xacro:property name="gripper_length" value="0.1"/>
   <material name="blue">
     <color rgba="0 0 1 1"/>
@@ -88,4 +89,32 @@
     </inertial>
   </link>
+  <link name="link_6">
+    <inertial>
+        <origin xyz="0 0 ${l5/2}" />
+        <mass value="1"/>
+        <inertia ixx="0.1" ixy="0" ixz="0" iyy="0.1" iyz="0" izz="0.1"/>
+      </inertial>
+      <visual>
+        <origin xyz="0 0 ${l5/2}" />
+        <geometry>
+          <box size="0.1 0.1 ${l5}" />
+      </geometry>
+      <material name="green" />
+    </visual>
+  </link>
+  <link name="gripper_link">
+    <visual>
+      <origin xyz="0 0 ${-gripper_length/2}" />
+      <geometry>
+        <box size="0.08 0.08 ${gripper_length}" />
+      </geometry>
+      <material name="red"/>
+    </visual>
+    <inertial>
+      <mass value="0.2"/>
+      <origin xyz="0 0 ${-gripper_length/2}" />
+      <inertia ixx="0.1" ixy="0" ixz="0" iyy="0.1" iyz="0" izz="0.1"/>
+    </inertial>
+  </link>
 <!--Joints-->
   <joint name="fixedjoint_1" type="fixed">
@@ -102,4 +131,9 @@
     <child link="link_5"/>
     <origin xyz="0 0 ${l4/2}"/>
+  </joint>
+  <joint name="gripper_joint" type="fixed">
+    <parent link="link_6"/>
+    <child link="gripper_link"/>
+    <origin xyz="0 0 0" />
   </joint>
 <!--revolut joints-->
@@ -120,3 +154,10 @@
     <dynamics damping="0.2" friction="0.1"/>
   </joint>
+  <joint name="prismatic_joint_1" type="prismatic">
+    <parent link="link_5" />
+    <child link="link_6" />
+    <origin xyz="${l5} 0 0" rpy="0 0 0" />
+    <axis xyz="0 0 1" />
+    <limit lower="0.0" upper="${-l5}" effort="100"  velocity="1.0" />
+  </joint>
 </robot>

Commit message: urdf update

File: test_1/urdf/scara_urdf.xacro (robot description, xacro)
@@ -6,5 +6,5 @@
   <xacro:property name="l4" value="0.2"/>
   <xacro:property name="l4_r" value="0.05"/>
-  <xacro:property name="l5" value="0.345"/>
+  <xacro:property name="l5" value="0.3"/>
   <xacro:property name="gripper_length" value="0.1"/>
   <material name="blue">
@@ -105,5 +105,5 @@
   <link name="gripper_link">
     <visual>
-      <origin xyz="0 0 ${-gripper_length/2}" />
+      <origin xyz="0 0 0" />
       <geometry>
         <box size="0.08 0.08 ${gripper_length}" />
@@ -113,5 +113,5 @@
     <inertial>
       <mass value="0.2"/>
-      <origin xyz="0 0 ${-gripper_length/2}" />
+      <origin xyz="0 0 0" />
       <inertia ixx="0.1" ixy="0" ixz="0" iyy="0.1" iyz="0" izz="0.1"/>
     </inertial>
@@ -135,5 +135,5 @@
     <parent link="link_6"/>
     <child link="gripper_link"/>
-    <origin xyz="0 0 0" />
+    <origin xyz="0 0 ${-gripper_length/2}" />
   </joint>
 <!--revolut joints-->
@@ -158,6 +158,6 @@
     <child link="link_6" />
     <origin xyz="${l5} 0 0" rpy="0 0 0" />
-    <axis xyz="0 0 1" />
-    <limit lower="0.0" upper="${-l5}" effort="100"  velocity="1.0" />
+    <axis xyz="0 0 -1" />
+    <limit lower="0.0" upper="${l5}" effort="100"  velocity="1.0" />
   </joint>
 </robot>
